Commit message: Add files via upload
Signed-off-by: SybilSystem001 <118040882+SybilSystem001@users.noreply.github.com>

File: open_manipulator_description/urdf/omx/omx.urdf.xacro (robot description, xacro)
@@ -7,7 +7,9 @@
   <xacro:arg name="port_name" default="/dev/ttyUSB0" />
   <xacro:arg name="ros2_control_type" default="omx" />
+  <xacro:property name="PI" value="3.14159274"/>
   <xacro:include filename="$(find open_manipulator_description)/gazebo/omx.gazebo.xacro" />
   <xacro:include filename="$(find open_manipulator_description)/urdf/omx/omx_arm.urdf.xacro" />
   <xacro:include filename="$(find open_manipulator_description)/ros2_control/$(arg ros2_control_type).ros2_control.xacro" />
+  <xacro:include filename="$(find open_manipulator_description)/urdf/camera/camera.xacro"/>
   <link name="world"/>
   <joint name="$(arg prefix)world_fixed" type="fixed">
@@ -23,4 +25,9 @@
     fake_sensor_commands="$(arg fake_sensor_commands)"
     port_name="$(arg port_name)"/>
+    <!-- Camera -->
+  <xacro:camera_v0 parent="world">
+    <origin xyz="0.2 0.6 0.7" rpy="0 ${PI/2} 0"/>
+  </xacro:camera_v0>
+  <xacro:camera_gazebo_v0/>
   <gazebo>
     <plugin filename="gz_ros2_control-system" name="gz_ros2_control::GazeboSimROS2ControlPlugin">

Commit message: added docker file for the turtlebot and changed the description of the open manipulator

File: open_manipulator_description/urdf/omx/omx.urdf.xacro (robot description, xacro)
@@ -27,5 +27,5 @@
     <!-- Camera -->
   <xacro:depthai_camera parent="link5">
-    <origin xyz="0.068 0 0.059" rpy="${PI/2} 0 ${PI/2}"/>
+    <origin xyz="0.061 0.028 0.059" rpy="${PI/2} 0 ${PI/2}"/>
   </xacro:depthai_camera>
   <xacro:camera_gazebo_v0/>

Commit message: added camera bracket to the model

File: open_manipulator_description/urdf/omx/omx.urdf.xacro (robot description, xacro)
@@ -26,6 +26,6 @@
     port_name="$(arg port_name)"/>
     <!-- Camera -->
-  <xacro:depthai_camera parent="link5">
-    <origin xyz="0.061 0.028 0.059" rpy="${PI/2} 0 ${PI/2}"/>
+  <xacro:depthai_camera parent="Camera_bracket">
+    <origin xyz="0.061 0.0445 0.097" rpy="${PI/2} 0 ${PI/2}"/>
   </xacro:depthai_camera>
   <xacro:camera_gazebo_v0/>

File: open_manipulator_description/urdf/omx/omx_arm.urdf.xacro (robot description, xacro)
@@ -157,4 +157,33 @@
       </inertial>
     </link>
+    <joint name="${prefix}Camera_joint" type="fixed">
+      <parent link="${prefix}link5"/>
+      <child link="${prefix}Camera_bracket"/>
+      <origin xyz="0.0 -0.0445 -0.025" rpy="0 0 0"/>
+    </joint>
+    <link name="${prefix}Camera_bracket">
+      <visual>
+        <origin xyz="0 0 0" rpy="0 0 0"/>
+        <geometry>
+          <mesh filename="${meshes_file_direction}/Camera_bracket.STL" scale="0.001 0.001 0.001"/>
+        </geometry>
+        <material name="grey">
+          <color rgba="0.2 0.2 0.2 1"/>
+        </material>
+      </visual>
+      <collision>
+        <origin xyz="0 0 0" rpy="0 0 0"/>
+        <geometry>
+          <mesh filename="${meshes_file_direction}/Camera_bracket.STL" scale="0.001 0.001 0.001"/>
+        </geometry>
+      </collision>
+       <inertial>
+        <origin xyz="4.4206755e-02 3.6839985e-07 8.9142216e-03" />
+        <mass value="1.4327573e-01" />
+        <inertia ixx="8.0870749e-05" ixy="0.0" ixz="-1.0157896e-06"
+                 iyy="7.5980465e-05" iyz="0.0"
+                 izz="9.3127351e-05" />
+      </inertial>
+    </link>
     <joint name="${prefix}gripper_left_joint" type="prismatic">
       <parent link="${prefix}link5"/>
