Commit message: changed end effector position

File: open_manipulator_description/urdf/omx/omx_arm.urdf.xacro (robot description, xacro)
@@ -254,5 +254,5 @@
       <parent link="${prefix}link5"/>
       <child link="${prefix}end_effector_link"/>
-      <origin xyz="0.126 0.0 0.0" rpy="0 0 0"/>
+      <origin xyz="0.125 0.0 0.0" rpy="0 0 0"/>
     </joint>
     <link name="${prefix}end_effector_link">
