Commit message: added oakd pro model

File: open_manipulator_description/urdf/camera/camera.xacro (robot description, xacro)
@@ -1,6 +1,6 @@
 <?xml version="1.0"?>
-<robot name="delirobo" xmlns:xacro="http://ros.org/wiki/xacro">
+<robot name="depthai_camera" xmlns:xacro="http://ros.org/wiki/xacro">
   <xacro:include filename="$(find open_manipulator_description)/urdf/camera/camera.gazebo"/>
-  <xacro:macro name="camera_v0" params="parent *joint_origin">
+  <xacro:macro name="depthai_camera" params="parent *joint_origin">
 	<joint name="camera_joint" type="fixed">
 	  <xacro:insert_block name="joint_origin"/>
@@ -10,7 +10,10 @@
 	<link name="camera_link">
 	  <visual>
-		<geometry>
-		  <mesh filename="package://open_manipulator_description/meshes/camera/visual/camera.dae"/>
-		</geometry>
+		  <geometry>
+		    <mesh filename="package://open_manipulator_description/meshes/camera/visual/camera.stl"/>
+		  </geometry>
+		<material name="black">
+      <color rgba="0 0 0 1"/>
+    </material>
 	  </visual>
 	  <collision>

File: open_manipulator_description/urdf/omx/omx.urdf.xacro (robot description, xacro)
@@ -26,12 +26,12 @@
     port_name="$(arg port_name)"/>
     <!-- Camera -->
-  <xacro:camera_v0 parent="world">
-    <origin xyz="0.2 0.6 0.7" rpy="0 ${PI/2} 0"/>
-  </xacro:camera_v0>
+  <xacro:depthai_camera parent="world">
+    <origin xyz="0.2 0.6 0.2" rpy="${PI/2} 0 ${PI/2}"/>
+  </xacro:depthai_camera>
   <xacro:camera_gazebo_v0/>
   <gazebo>
     <plugin filename="gz_ros2_control-system" name="gz_ros2_control::GazeboSimROS2ControlPlugin">
-      <!-- <parameters>$(find open_manipulator_bringup)/config/omx/hardware_controller_manager.yaml</parameters> -->
-      <parameters>$(find open_manipulator_bringup)/config/omx/gazebo_controller_manager.yaml</parameters>
+      <parameters>$(find open_manipulator_bringup)/config/omx/hardware_controller_manager.yaml</parameters>
+      <!--  <parameters>$(find open_manipulator_bringup)/config/omx/gazebo_controller_manager.yaml</parameters> -->
     </plugin>
   </gazebo>

Commit message: camera now attached to link5

File: open_manipulator_description/urdf/camera/camera.xacro (robot description, xacro)
@@ -14,5 +14,5 @@
 		  </geometry>
 		<material name="black">
-      <color rgba="0 0 0 1"/>
+      <color rgba="0.05 0.05 0.05 1"/>
     </material>
 	  </visual>

File: open_manipulator_description/urdf/omx/omx.urdf.xacro (robot description, xacro)
@@ -26,6 +26,6 @@
     port_name="$(arg port_name)"/>
     <!-- Camera -->
-  <xacro:depthai_camera parent="world">
-    <origin xyz="0.2 0.6 0.2" rpy="${PI/2} 0 ${PI/2}"/>
+  <xacro:depthai_camera parent="link5">
+    <origin xyz="0.068 0 0.059" rpy="${PI/2} 0 ${PI/2}"/>
   </xacro:depthai_camera>
   <xacro:camera_gazebo_v0/>

Commit message: added new collision awareness and changed initial position

File: open_manipulator_description/urdf/camera/camera.xacro (robot description, xacro)
@@ -24,5 +24,5 @@
 	  <inertial>
 		<origin xyz="0 0 0"/>
-		<mass value="0.1"/>
+		<mass value="0.091"/>
 		<inertia ixx="0.00001" ixy="0" ixz="0" iyy="0.00001" iyz="0" izz="0.00001" />
 	  </inertial>
